File: pcb/mastertemp_esp32/mastertemp_esp32.kicad_pcb (KiCad board)
At the start: 4 copper layers, 160 x 100 mm, 0 parts

Commit message: Starting design
Other:
- board text added: "AC OPTO SENSE FIELD SIDE LEFT"
- board text added: "D1 / TVS / BULK VRAW"
- board text added: "ESP32 ANTENNA KEEPOUT"
- board text added: "FUTURE ISOLATION SLOT"
- board text added: "ICM REF S1/240 S1/120 L1 L2 S2 TH IND VAL GND"
- board text added: "INSTALL/SERVICE BY QUALIFIED TECHNICIAN"
- board text added: "J1 POWER 3P 24 VAC CLASS II ONLY"
- board text added: "J2 OPERATING CONTROL 7P VAL TH IND GND 24VAC 24VAC FS"
- board text added: "J3 SAFETY STACK 7P PS HLS ES1 AFS AGS SFS GAS"
- board text added: "J4 THERM 2P"
- board text added: "J5 EXT CTRL 3P SPA COMMON POOL"
- board text added: "J6 MEMBRANE / UI 12P"
- board text added: "J6 SERVICE UART"
- board text added: "K1 NO RELAY"
- board text added: "K2 NO RELAY"
- board text added: "NO COPPER / NO PARTS"
- board text added: "SERIES TH PATH - WIDE CLEARANCE"
- board text added: "TP ROW: VRAW +5V +3V3 WDG SAFETY K1 K2 TH VAL"
- board text added: "U1/L1 100 V BUCK COMPACT HOT LOOP"
- board text added: "U3/U4/U6 SUPERVISOR + IO"
- board text added: "U5 ESP32-WROOM ANTENNA TOWARD EDGE"
- board text added: "U7 ADC / U16-U17 QUIET ANALOG"
- board text added: "VAL / GAS MONITOR ONLY - NO DRIVE"
- board text added: "ZONE A: 24 VAC INPUT / PROTECTION"
- board text added: "ZONE B: VRAW BUCK"
- board text added: "ZONE C: ESP32 / LOGIC / ADC"
- board text added: "ZONE D: ICM + SERIES TH RELAYS"
- board text added: "ZONE E: SAFETY / REMOTE / UI"

Commit message: Bump
Parts:
- added C1: 470uF_63V, CP_Radial_D10.0mm_P5.00mm, F.Cu at (73.0, 47.0)
- added D1: MB10S, SOIC-4_4.55x3.7mm_P2.54mm, F.Cu at (48.0, 47.0)
- added F1: 0.5A_FUSE, Fuse_1206_3216Metric, F.Cu at (29.0, 47.0)
- added J1: 24VAC_IN, PhoenixContact_MSTBA_2,5_3-G-5,08_1x03_P5.08mm_Horizontal, F.Cu at (34.0, 34.0)
- added J2: OPERATING_CONTROL, PhoenixContact_MSTBA_2,5_7-G-5,08_1x07_P5.08mm_Horizontal, F.Cu at (44.0, 104.0)
- added J3: SAFETY_STACK, PhoenixContact_MSTBA_2,5_7-G-5,08_1x07_P5.08mm_Horizontal, F.Cu at (84.0, 104.0)
- added J4: THERMISTOR, PhoenixContact_MSTBA_2,5_2-G-5,08_1x02_P5.08mm_Horizontal, F.Cu at (132.0, 104.0)
- added J5: EXT_CONTROL, PhoenixContact_MSTBA_2,5_3-G-5,08_1x03_P5.08mm_Horizontal, F.Cu at (160.0, 104.0)
- added J6: MEMBRANE_REF, PhoenixContact_MSTBA_2,5_9-G-5,08_1x09_P5.08mm_Horizontal, F.Cu at (135.0, 84.0)
- added K1: G5Q-1A-DC5, Relay_SPST_Omron-G5Q-1A, F.Cu at (43.0, 88.0)
- added K2: G5Q-1A-DC5, Relay_SPST_Omron-G5Q-1A, F.Cu at (66.0, 88.0)
- added L1: 68uH, L_12x12mm_H8mm, F.Cu at (70.0, 66.0)
- added L2: 2.2uH, L_Vishay_IFSC-1515AH_4x4x1.8mm, F.Cu at (103.0, 66.0)
- added MOV1: V47ZA1P, RV_Disc_D7mm_W3.9mm_P5mm, F.Cu at (37.0, 47.0)
- added Q1: AO3400A, SOT-23, F.Cu at (34.0, 96.0)
- added Q2: AO3400A, SOT-23, F.Cu at (78.0, 96.0)
- added TP1: VRAW, TestPoint_Pad_D2.0mm, F.Cu at (98.0, 36.0)
- added TP2: +5V, TestPoint_Pad_D2.0mm, F.Cu at (106.0, 36.0)
- added TP3: +3V3, TestPoint_Pad_D2.0mm, F.Cu at (114.0, 36.0)
- added TP4: WATCHDOG_OK, TestPoint_Pad_D2.0mm, F.Cu at (122.0, 36.0)
- added TP5: SAFETY_STATIC_OK, TestPoint_Pad_D2.0mm, F.Cu at (126.0, 36.0)
- added TP6: K1_COIL, TestPoint_Pad_D2.0mm, F.Cu at (98.0, 43.0)
- added TP7: K2_COIL, TestPoint_Pad_D2.0mm, F.Cu at (106.0, 43.0)
- added TP8: TH_FEEDBACK, TestPoint_Pad_D2.0mm, F.Cu at (114.0, 43.0)
- added TP9: VAL_SENSE, TestPoint_Pad_D2.0mm, F.Cu at (122.0, 43.0)
- added TVS1: SMBJ51CA, D_SMB, F.Cu at (63.0, 47.0)
- added U1: LM5164YDRCR, Texas_S-PVSON-N10, F.Cu at (55.0, 66.0)
- added U10: H11AA1M_IND, DIP-6_W7.62mm, F.Cu at (31.0, 69.0)
- added U11: H11AA1M_VAL, DIP-6_W7.62mm, F.Cu at (41.0, 56.0)
- added U12: H11AA1M_24VAC, DIP-6_W7.62mm, F.Cu at (41.0, 69.0)
- added U16: TLV6700DDCR_THERM, SOT-23-6, F.Cu at (124.0, 75.0)
- added U17: TLV6700DDCR_SFS, SOT-23-6, F.Cu at (124.0, 83.0)
- added U18: OPA333AIDBVR, SOT-23-5, F.Cu at (134.0, 78.0)
- added U2: AP63203WU-7, TSOT-23-6, F.Cu at (95.0, 66.0)
- added U3: TPS3839G33DBZR, SOT-23-3, F.Cu at (110.0, 48.0)
- added U4: TPS3823-33DBVR, SOT-23-5, F.Cu at (120.0, 48.0)
- added U5: ESP32-WROOM-32E-N16, ESP32-WROOM-32E, F.Cu at (153.0, 55.0)
- added U6: MCP23017-E/SS, SSOP-28_5.3x10.2mm_P0.65mm, F.Cu at (114.0, 61.0)
- added U7: ADS1115IDGSR, VSSOP-10_3x3mm_P0.5mm, F.Cu at (114.0, 78.0)
- added U8: NXE1S0505MC-R7, Converter_DCDC_Murata_NXExSxxxxMC_SMD, F.Cu at (95.0, 87.0)
- added U9: H11AA1M_TH, DIP-6_W7.62mm, F.Cu at (31.0, 56.0)
Routing:
- net TH_HEAT_REQUEST_OUT: track 0.00 -> 55.4 mm
- net ICM_24VAC_SOURCE: track 0.00 -> 27.2 mm
- net HEAT_CHAIN_K1_K2: track 0.00 -> 23.4 mm
Other:
- board text added: "J6 MEMBRANE REF 9P KEYPAD OUT OF SCOPE"
- board text removed: "J6 MEMBRANE / UI 12P"

Commit message: AI
Parts:
- added C10: SFS_ADC_FILTER_TBD, Capacitor_SMD:C_0805_2012Metric, F.Cu at (138.0, 75.0)
- added C11: VRAW_MON_FILTER_TBD, Capacitor_SMD:C_0805_2012Metric, F.Cu at (134.0, 72.5)
- added C2: 100nF_REMOTE_FILTER_TBD, Capacitor_SMD:C_0805_2012Metric, F.Cu at (116.0, 91.0)
- added C3: 100nF_REMOTE_FILTER_TBD, Capacitor_SMD:C_0805_2012Metric, F.Cu at (127.0, 91.0)
- added C4: 2.2uF_100V_VRAW_IN_TBD, Capacitor_SMD:C_1210_3225Metric, F.Cu at (55.0, 60.0)
- added C5: 2.2nF_50V_BST_5V, Capacitor_SMD:C_0603_1608Metric, F.Cu at (61.0, 62.0)
- added C6: 100nF_BST_3V3, Capacitor_SMD:C_0603_1608Metric, F.Cu at (98.5, 66.0)
- added C7: 10uF_50V_3V3_IN_TBD, Capacitor_SMD:C_1210_3225Metric, F.Cu at (95.0, 70.0)
- added C8: 22uF_10V_3V3_OUT_TBD, Capacitor_SMD:C_0805_2012Metric, F.Cu at (107.0, 70.0)
- added C9: THERM_ADC_FILTER_TBD, Capacitor_SMD:C_0805_2012Metric, F.Cu at (157.0, 86.0)
- added D2: K1_FLYBACK_TBD, Diode_SMD:D_SOD-123, F.Cu at (38.0, 84.0)
- added D3: K2_FLYBACK_TBD, Diode_SMD:D_SOD-123, F.Cu at (70.0, 76.0)
- added R1: 2.2k_REMOTE_WET_TBD, Resistor_SMD:R_0805_2012Metric, F.Cu at (116.0, 100.0)
- added R10: K1_GATE_PULLDOWN_TBD, Resistor_SMD:R_0805_2012Metric, F.Cu at (30.5, 101.5)
- added R11: K2_GATE_PULLDOWN_TBD, Resistor_SMD:R_0805_2012Metric, F.Cu at (70.5, 98.5)
- added R12: VAL_OPTO_PULLUP_TBD, Resistor_SMD:R_0805_2012Metric, F.Cu at (124.5, 50.0)
- added R13: TH_OPTO_LIMIT_A_TBD, Resistor_SMD:R_0805_2012Metric, F.Cu at (22.0, 56.0)
- added R14: TH_OPTO_LIMIT_B_TBD, Resistor_SMD:R_0805_2012Metric, F.Cu at (26.0, 56.0)
- added R15: TH_OPTO_PULLUP_TBD, Resistor_SMD:R_0805_2012Metric, F.Cu at (130.5, 50.0)
- added R16: IND_OPTO_LIMIT_A_TBD, Resistor_SMD:R_0805_2012Metric, F.Cu at (24.0, 69.0)
- added R17: IND_OPTO_LIMIT_B_TBD, Resistor_SMD:R_0805_2012Metric, F.Cu at (28.0, 69.0)
- added R18: IND_OPTO_PULLUP_TBD, Resistor_SMD:R_0805_2012Metric, F.Cu at (136.5, 50.0)
- added R19: VAC24_OPTO_LIMIT_A_TBD, Resistor_SMD:R_0805_2012Metric, F.Cu at (32.0, 78.0)
- added R2: 2.2k_REMOTE_WET_TBD, Resistor_SMD:R_0805_2012Metric, F.Cu at (127.0, 100.0)
- added R20: VAC24_OPTO_LIMIT_B_TBD, Resistor_SMD:R_0805_2012Metric, F.Cu at (28.0, 78.0)
- added R21: VAC24_OPTO_PULLUP_TBD, Resistor_SMD:R_0805_2012Metric, F.Cu at (136.5, 54.0)
- added R22: K1_GATE_SERIES_TBD, Resistor_SMD:R_0805_2012Metric, F.Cu at (26.0, 98.0)
- added R23: K2_GATE_SERIES_TBD, Resistor_SMD:R_0805_2012Metric, F.Cu at (68.0, 95.0)
- added R24: THERM_PULLUP_TBD, Resistor_SMD:R_0805_2012Metric, F.Cu at (153.0, 86.0)
- added R25: I2C_SDA_PULLUP_TBD, Resistor_SMD:R_0805_2012Metric, F.Cu at (103.0, 58.8)
- added R26: I2C_SCL_PULLUP_TBD, Resistor_SMD:R_0805_2012Metric, F.Cu at (103.0, 56.0)
- added R27: SFS_INPUT_SERIES_TBD, Resistor_SMD:R_0805_2012Metric, F.Cu at (130.0, 77.0)
- added R28: VRAW_MON_TOP_TBD, Resistor_SMD:R_0805_2012Metric, F.Cu at (101.0, 40.0)
- added R29: VRAW_MON_BOT_TBD, Resistor_SMD:R_0805_2012Metric, F.Cu at (134.0, 70.0)
- added R3: 10k_REMOTE_PULLUP, Resistor_SMD:R_0805_2012Metric, F.Cu at (116.0, 88.0)
- added R30: THERM_RANGE_OK_PULLUP_TBD, Resistor_SMD:R_0805_2012Metric, F.Cu at (128.0, 74.0)
- added R31: SFS_RANGE_OK_PULLUP_TBD, Resistor_SMD:R_0805_2012Metric, F.Cu at (132.0, 84.0)
- added R32: THERM_LOW_REF_TOP_TBD, Resistor_SMD:R_0805_2012Metric, F.Cu at (162.0, 82.0)
- added R33: THERM_LOW_REF_BOT_TBD, Resistor_SMD:R_0805_2012Metric, F.Cu at (166.0, 82.0)
- added R34: THERM_HIGH_REF_TOP_TBD, Resistor_SMD:R_0805_2012Metric, F.Cu at (162.0, 88.0)
- added R35: THERM_HIGH_REF_BOT_TBD, Resistor_SMD:R_0805_2012Metric, F.Cu at (166.0, 88.0)
- added R36: SFS_LOW_REF_TOP_TBD, Resistor_SMD:R_0805_2012Metric, F.Cu at (162.0, 90.0)
- added R37: SFS_LOW_REF_BOT_TBD, Resistor_SMD:R_0805_2012Metric, F.Cu at (166.0, 90.0)
- added R38: SFS_HIGH_REF_TOP_TBD, Resistor_SMD:R_0805_2012Metric, F.Cu at (162.0, 94.0)
- added R39: SFS_HIGH_REF_BOT_TBD, Resistor_SMD:R_0805_2012Metric, F.Cu at (166.0, 94.0)
- added R4: 10k_REMOTE_PULLUP, Resistor_SMD:R_0805_2012Metric, F.Cu at (127.0, 88.0)
- added R5: RFB5V_TOP_TBD, Resistor_SMD:R_0805_2012Metric, F.Cu at (61.0, 70.0)
- added R6: RFB5V_BOT_TBD, Resistor_SMD:R_0805_2012Metric, F.Cu at (61.0, 73.0)
- added R7: RON5V_TBD, Resistor_SMD:R_0805_2012Metric, F.Cu at (55.0, 72.0)
- added R8: VAL_OPTO_LIMIT_A_TBD, Resistor_SMD:R_0805_2012Metric, F.Cu at (24.0, 64.0)
- added R9: VAL_OPTO_LIMIT_B_TBD, Resistor_SMD:R_0805_2012Metric, F.Cu at (29.0, 64.0)
- added U14: THERMISTOR_AFE_TBD, Package_TO_SOT_SMD:SOT-23-6, F.Cu at (148.0, 82.0)
- added U19: LTV-817S_SPA_CANDIDATE, Package_DIP:DIP-4_W7.62mm, F.Cu at (116.0, 94.0)
- added U20: LTV-817S_POOL_CANDIDATE, Package_DIP:DIP-4_W7.62mm, F.Cu at (127.0, 94.0)
- C1: footprint CP_Radial_D10.0mm_P5.00mm -> Capacitor_THT:CP_Radial_D10.0mm_P5.00mm
- D1: footprint SOIC-4_4.55x3.7mm_P2.54mm -> Diode_SMD:Diode_Bridge_Vishay_MBLS
- F1: footprint Fuse_1206_3216Metric -> Fuse:Fuse_1206_3216Metric
- J1, J5: footprint PhoenixContact_MSTBA_2,5_3-G-5,08_1x03_P5.08mm_Horizontal -> Connector_Phoenix_MSTB:PhoenixContact_MSTBA_2,5_3-G-5,08_1x03_P5.08mm_Horizontal
- J2, J3: footprint PhoenixContact_MSTBA_2,5_7-G-5,08_1x07_P5.08mm_Horizontal -> Connector_Phoenix_MSTB:PhoenixContact_MSTBA_2,5_7-G-5,08_1x07_P5.08mm_Horizontal
- J4: footprint PhoenixContact_MSTBA_2,5_2-G-5,08_1x02_P5.08mm_Horizontal -> Connector_Phoenix_MSTB:PhoenixContact_MSTBA_2,5_2-G-5,08_1x02_P5.08mm_Horizontal
- J6: footprint PhoenixContact_MSTBA_2,5_9-G-5,08_1x09_P5.08mm_Horizontal -> Connector_Phoenix_MSTB:PhoenixContact_MSTBVA_2,5_9-G-5,08_1x09_P5.08mm_Vertical
- K1, K2: footprint Relay_SPST_Omron-G5Q-1A -> Relay_THT:Relay_SPST_Omron-G5Q-1A
- L1: footprint L_12x12mm_H8mm -> Inductor_SMD:L_12x12mm_H8mm
- L2: footprint L_Vishay_IFSC-1515AH_4x4x1.8mm -> Inductor_SMD:L_Vishay_IFSC-1515AH_4x4x1.8mm
- MOV1: footprint RV_Disc_D7mm_W3.9mm_P5mm -> Varistor:RV_Disc_D7mm_W3.9mm_P5mm
- Q1, Q2: footprint SOT-23 -> Package_TO_SOT_SMD:SOT-23
- TVS1: footprint D_SMB -> Diode_SMD:D_SMB
- U1: value LM5164YDRCR -> LM5164DDAR; footprint Texas_S-PVSON-N10 -> Package_SO:TI_SO-PowerPAD-8
- U10, U11, U12, U9: footprint DIP-6_W7.62mm -> Package_DIP:DIP-6_W7.62mm
- U16, U17: footprint SOT-23-6 -> Package_TO_SOT_SMD:SOT-23-6
- U18, U4: footprint SOT-23-5 -> Package_TO_SOT_SMD:SOT-23-5
- U2: footprint TSOT-23-6 -> Package_TO_SOT_SMD:TSOT-23-6
- U3: footprint SOT-23-3 -> Package_TO_SOT_SMD:SOT-23-3
- U6: footprint SSOP-28_5.3x10.2mm_P0.65mm -> Package_SO:SSOP-28_5.3x10.2mm_P0.65mm
- U7: footprint VSSOP-10_3x3mm_P0.5mm -> Package_SO:VSSOP-10_3x3mm_P0.5mm
- U8: footprint Converter_DCDC_Murata_NXExSxxxxMC_SMD -> Converter_DCDC:Converter_DCDC_Murata_NXExSxxxxMC_SMD
- moved TP6 80.7 mm to (31.0, 88.0)
- moved TP7 55.5 mm to (82.0, 93.0)
- moved J6 42.7 mm to (176.0, 96.0), turned to 90 degrees
- moved D1 6.71 mm to (54.0, 50.0)
Connections:
- net EARTH_SHIELD_REF renamed CHASSIS_SHIELD
- C1 pad 1: (no net) -> VRAW
- C1 pad 2: (no net) -> PGND_RAW
- D1 pad 1: (no net) -> VAC24_A_FUSED
- D1 pad 3: (no net) -> VRAW
- D1 pad 4: (no net) -> PGND_RAW
- F1 pad 1: (no net) -> VAC24_A_FUSED
- F1 pad 2: (no net) -> VAC24_A
- J1 pad 1: 24VAC_A -> VAC24_A
- J1 pad 2: 24VAC_B -> VAC24_B
- L1 pad 1: (no net) -> SW_5V
- L1 pad 2: (no net) -> +5V
- MOV1 pad 1: (no net) -> VAC24_A_FUSED
- MOV1 pad 2: (no net) -> VAC24_B
- TVS1 pad 1: (no net) -> VAC24_A_FUSED
- TVS1 pad 2: (no net) -> VAC24_B
- U1 pad 1: (no net) -> PGND_RAW
- U1 pad 2: (no net) -> VRAW
- U1 pad 3: (no net) -> VRAW
- U1 pad 4: (no net) -> RON_5V_TBD
- U1 pad 5: (no net) -> FB_5V_TBD
- U1 pad 6: (no net) -> +5V_PGOOD
- U1 pad 7: (no net) -> BST_5V
- U1 pad 8: (no net) -> SW_5V
- U1 pad 9: (no net) -> PGND_RAW
- U10 pad 1: (no net) -> IND_OPTO_INPUT
- U10 pad 2: (no net) -> ICM_GND_REF
- U10 pad 4: (no net) -> GND
- U10 pad 5: (no net) -> IND_OPTO_GPIO
- U11 pad 1: (no net) -> VAL_OPTO_INPUT
- U11 pad 2: (no net) -> ICM_GND_REF
- U11 pad 4: (no net) -> GND
- U11 pad 5: (no net) -> VAL_OPTO_GPIO
- U12 pad 1: (no net) -> VAC24_OPTO_INPUT
- U12 pad 2: (no net) -> ICM_GND_REF
- U12 pad 4: (no net) -> GND
- U12 pad 5: (no net) -> VAC24_OPTO_GPIO
- U16 pad 1: (no net) -> THERM_WINDOW_SENSE
- U16 pad 2: (no net) -> THERM_LOW_REF_TBD
- U16 pad 3: (no net) -> THERM_HIGH_REF_TBD
- U16 pad 4: (no net) -> THERMISTOR_RANGE_OK
- U16 pad 5: (no net) -> GND
- U17 pad 1: (no net) -> SFS_WINDOW_SENSE
- U17 pad 2: (no net) -> SFS_LOW_REF_TBD
- U17 pad 3: (no net) -> SFS_HIGH_REF_TBD
- U17 pad 4: (no net) -> SFS_RANGE_OK
- U17 pad 5: (no net) -> GND
- U18 pad 1: (no net) -> SFS_FIELD_INPUT
- U18 pad 2: (no net) -> SFS_RETURN_OR_REF
- U18 pad 3: (no net) -> +3V3_ADC
- U18 pad 4: (no net) -> AGND
- U18 pad 5: (no net) -> SFS_ADC
- U2 pad 1: (no net) -> +3V3
- U2 pad 2: GND -> +5V
- U2 pad 3: (no net) -> +5V
- U2 pad 4: (no net) -> SW_3V3
- U2 pad 5: +5V -> GND
- U2 pad 6: SW_3V3 -> BST_3V3
- U3 pad 1: ESP32_EN -> BROWNOUT_OK
- U6 pad 10: (no net) -> GND
- U6 pad 12: (no net) -> I2C_SCL
- U6 pad 13: (no net) -> I2C_SDA
- U6 pad 15: (no net) -> GND
- U6 pad 16: (no net) -> GND
- U6 pad 17: (no net) -> GND
- U6 pad 18: (no net) -> +3V3
- U6 pad 21: (no net) -> VAL_OPTO_GPIO
- U6 pad 22: (no net) -> TH_OPTO_GPIO
- U6 pad 23: (no net) -> IND_OPTO_GPIO
- U6 pad 24: (no net) -> VAC24_OPTO_GPIO
- U6 pad 9: (no net) -> +3V3
- U7 pad 8: TH_FEEDBACK_ADC -> VRAW_MONITOR_ADC
- U8 pad 1: (no net) -> GND
- U8 pad 3: (no net) -> +5V
- U8 pad 7: (no net) -> COMMON_LINE
- U8 pad 8: (no net) -> ISO_REMOTE_5V
- U9 pad 1: (no net) -> TH_OPTO_INPUT
- U9 pad 2: (no net) -> ICM_GND_REF
- U9 pad 4: (no net) -> GND
- U9 pad 5: (no net) -> TH_OPTO_GPIO
Routing:
- net GND: track 0.00 -> 475.0 mm, vias 0 -> 16
- net +3V3: track 0.00 -> 278.0 mm
- net VAL_SENSE_AC: track 0.00 -> 225.1 mm, vias 0 -> 2
- net IND_OPTO_GPIO: track 0.00 -> 173.5 mm, vias 0 -> 3
- net VAC24_OPTO_GPIO: track 0.00 -> 169.1 mm, vias 0 -> 3
- net SFS_INPUT: track 0.00 -> 162.6 mm, vias 0 -> 1
- net TH_OPTO_GPIO: track 0.00 -> 159.2 mm, vias 0 -> 2
- net VAL_OPTO_GPIO: track 0.00 -> 151.7 mm, vias 0 -> 2
- net COMMON_LINE: track 0.00 -> 137.8 mm, vias 0 -> 1
- net ICM_GND_REF: track 0.00 -> 121.6 mm
- net +5V: track 0.00 -> 110.2 mm, vias 0 -> 2
- net SFS_ADC: track 0.00 -> 103.0 mm, vias 0 -> 2
- net VRAW_MONITOR_ADC: track 0.00 -> 97.1 mm, vias 0 -> 3
- net AGND: track 0.00 -> 96.9 mm, vias 0 -> 4
- net VRAW: track 0.00 -> 87.5 mm
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Other:
- board text added: "GAS MONITOR ONLY - NO DRIVE"
- board text added: "NO LINE VOLTAGE"
