File: pcb/mastertemp_esp32/sheets/esp32_supervisor.kicad_sch (KiCad schematic)
At the start: 0 parts

Commit message: Make open source.
Parts:
- added TPI2CSCL: I2C_SCL_REVIEW_STUB, symbol mastertemp_esp32:NetStub_1pin
- added TPI2CSDA: I2C_SDA_REVIEW_STUB, symbol mastertemp_esp32:NetStub_1pin
- added U4: WATCHDOG_SUPERVISOR_TBD, Package_TO_SOT_SMD:SOT-23-5, symbol mastertemp_esp32:Watchdog_4pin
- added U5: ESP32-WROOM-32E-N16_CANDIDATE, RF_Module:ESP32-WROOM-32, symbol mastertemp_esp32:ESP32_ControlBlock
- added U9: RELAY_GATE_LOGIC_TBD, symbol mastertemp_esp32:RelayGateLogic
Connections:
- new net +3V3: U4.1 (+3V3), U5.1 (+3V3)
- new net BROWNOUT_OK: U5.3 (ESP32_EN), U9.3 (BROWNOUT_OK)
- new net GND: U4.2 (GND), U5.2 (GND)
- new net HEAT_CMD_GPIO: U5.4 (HEAT_CMD_GPIO), U9.1 (HEAT_CMD_GPIO)
- new net I2C_SCL: TPI2CSCL.1 (NET), U5.8 (I2C_SCL)
- new net I2C_SDA: TPI2CSDA.1 (NET), U5.7 (I2C_SDA)
- new net NOT_OTA_FAULT: U5.6 (NOT_OTA_FAULT), U9.5 (NOT_OTA_FAULT)
- new net RELAY_K1_GATE: U9.6 (RELAY_K1_GATE)
- new net RELAY_K2_GATE: U9.7 (RELAY_K2_GATE)
- new net SAFETY_STATIC_OK: U9.4 (SAFETY_STATIC_OK)
- new net WATCHDOG_OK: U4.4 (WATCHDOG_OK), U9.2 (WATCHDOG_OK)
- new net WDI_HEARTBEAT: U4.3 (WDI), U5.5 (WDI_HEARTBEAT)
Other:
- note added: "ESP32 pins are placeholders from the preliminary design. Avoid strapping pins for relay commands; relay gates must default low."
- note added: "Relay gates are generated only from HEAT_CMD_GPIO, WATCHDOG_OK, BROWNOUT_OK, SAFETY_STATIC_OK, and NOT_OTA_FAULT. Final physical gate family, polarity, pull-downs, and reset behavior still require detailed capture and review."
- note added: "SCHEMATIC PASS 1 - ESP32 SUPERVISOR AND RELAY GATE CONTRACT"
- note removed: "TODO: ESP32-WROOM, watchdog, reset supervisor, programming header, I2C, relay-enable logic."
Changed lines of the file:
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@@
   (title_block
     (title "ESP32, Watchdog, Reset, Relay Enable Gates")
-    (date "2026-05-31")
-    (rev "scaffold-0")
+    (date "2026-06-01")
+    (rev "schematic-pass-1")
     (company "Preliminary - not certified")
     (comment 1 "Relay command pins must default off during reset, bootloader, brownout, OTA, and crash.")
   )
-  (text "TODO: ESP32-WROOM, watchdog, reset supervisor, programming header, I2C, relay-enable logic."
+  (text "SCHEMATIC PASS 1 - ESP32 SUPERVISOR AND RELAY GATE CONTRACT"
     (at 25.4 25.4 0)
-    (effects (font (size 1.5 1.5)) (justify left bottom))
+    (effects (font (size 1.8 1.8) (bold yes)) (justify left bottom))
+  )
+  (text "Relay gates are generated only from HEAT_CMD_GPIO, WATCHDOG_OK, BROWNOUT_OK, SAFETY_STATIC_OK, and NOT_OTA_FAULT.\nFinal physical gate family, polarity, pull-downs, and reset behavior still require detailed capture and review."
+    (at 25.4 35.56 0)
+    (effects (font (size 1.35 1.35)) (justify left top))
+  )
+  (text "ESP32 pins are placeholders from the preliminary design. Avoid strapping pins for relay commands; relay gates must default low."
+    (at 25.4 55.88 0)
+    (effects (font (size 1.35 1.35)) (justify left top))
+  )
+  (symbol
+    (lib_id "mastertemp_esp32:ESP32_ControlBlock")
+    (at 60.96 82.55 0)
+    (unit 1)
+    (exclude_from_sim no)
+    (in_bom yes)
+    (on_board yes)
+    (dnp no)
+    (property "Reference" "U5" (at 60.96 67.31 0) (effects (font (size 1.27 1.27))))
+    (property "Value" "ESP32-WROOM-32E-N16_CANDIDATE" (at 60.96 97.79 0) (effects (font (size 1.27 1.27))))
+    (property "Footprint" "RF_Module:ESP32-WROOM-32" (at 60.96 82.55 0) (effects (font (size 1.27 1.27)) (hide yes)))
+    (property "Datasheet" "~" (at 60.96 82.55 0) (effects (font (size 1.27 1.27)) (hide yes)))
+    (property "Description" "ESP32 control block placeholder" (at 60.96 82.55 0) (effects (font (size 1.27 1.27)) (hide yes)))
+    (pin "1")
+    (pin "2")
+    (pin "3")
+    (pin "4")
+    (pin "5")
+    (pin "6")
+    (pin "7")
+    (pin "8")
+    (instances (project "mastertemp_esp32" (path "/55f88e14-a963-4749-b9bf-a5d12f0d95cb" (reference "U5") (unit 1))))
+  )
+  (symbol
+    (lib_id "mastertemp_esp32:Watchdog_4pin")
+    (at 60.96 116.84 0)
+    (unit 1)
+    (exclude_from_sim no)
+    (in_bom yes)
+    (on_board yes)
+    (dnp no)
+    (property "Reference" "U4" (at 60.96 106.68 0) (effects (font (size 1.27 1.27))))
+    (property "Value" "WATCHDOG_SUPERVISOR_TBD" (at 60.96 127.0 0) (effects (font (size 1.27 1.27))))
+    (property "Footprint" "Package_TO_SOT_SMD:SOT-23-5" (at 60.96 116.84 0) (effects (font (size 1.27 1.27)) (hide yes)))
+    (property "Datasheet" "~" (at 60.96 116.84 0) (effects (font (size 1.27 1.27)) (hide yes)))
+    (property "Description" "External watchdog supervisor placeholder" (at 60.96 116.84 0) (effects (font (size 1.27 1.27)) (hide yes)))
+    (pin "1")
+    (pin "2")
+    (pin "3")
+    (pin "4")
+    (instances (project "mastertemp_esp32" (path "/55f88e14-a963-4749-b9bf-a5d12f0d95cb" (reference "U4") (unit 1))))
+  )
+  (symbol
+    (lib_id "mastertemp_esp32:RelayGateLogic")
+    (at 129.54 91.44 0)
+    (unit 1)
+    (exclude_from_sim no)
+    (in_bom yes)
+    (on_board yes)
+    (dnp no)
+    (property "Reference" "U9" (at 129.54 77.47 0) (effects (font (size 1.27 1.27))))
+    (property "Value" "RELAY_GATE_LOGIC_TBD" (at 129.54 105.41 0) (effects (font (size 1.27 1.27))))
+    (property "Footprint" "" (at 129.54 91.44 0) (effects (font (size 1.27 1.27)) (hide yes)))
+    (property "Datasheet" "~" (at 129.54 91.44 0) (effects (font (size 1.27 1.27)) (hide yes)))
+    (property "Description" "Relay enable logic placeholder; final gates and polarity TBD" (at 129.54 91.44 0) (effects (font (size 1.27 1.27)) (hide yes)))
+    (pin "1")
+    (pin "2")
+    (pin "3")
+    (pin "4")
+    (pin "5")
+    (pin "6")
+    (pin "7")
+    (instances (project "mastertemp_esp32" (path "/55f88e14-a963-4749-b9bf-a5d12f0d95cb" (reference "U9") (unit 1))))
+  )
+  (label "+3V3" (at 49.53 74.93 0) (fields_autoplaced yes) (effects (font (size 1.27 1.27)) (justify left bottom)))
+  (label "GND" (at 49.53 77.47 0) (fields_autoplaced yes) (effects (font (size 1.27 1.27)) (justify left bottom)))
+  (global_label "BROWNOUT_OK" (shape input) (at 49.53 80.01 0) (fields_autoplaced yes) (effects (font (size 1.27 1.27)) (justify left bottom)))
+  (label "HEAT_CMD_GPIO" (at 72.39 74.93 0) (fields_autoplaced yes) (effects (font (size 1.27 1.27)) (justify left bottom)))
+  (label "WDI_HEARTBEAT" (at 72.39 77.47 0) (fields_autoplaced yes) (effects (font (size 1.27 1.27)) (justify left bottom)))
+  (label "NOT_OTA_FAULT" (at 72.39 80.01 0) (fields_autoplaced yes) (effects (font (size 1.27 1.27)) (justify left bottom)))
+  (label "I2C_SDA" (at 72.39 82.55 0) (fields_autoplaced yes) (effects (font (size 1.27 1.27)) (justify left bottom)))
+  (label "I2C_SCL" (at 72.39 85.09 0) (fields_autoplaced yes) (effects (font (size 1.27 1.27)) (justify left bottom)))
+  (label "+3V3" (at 52.07 113.03 0) (fields_autoplaced yes) (effects (font (size 1.27 1.27)) (justify left bottom)))
+  (label "GND" (at 52.07 115.57 0) (fields_autoplaced yes) (effects (font (size 1.27 1.27)) (justify left bottom)))
+  (label "WDI_HEARTBEAT" (at 52.07 118.11 0) (fields_autoplaced yes) (effects (font (size 1.27 1.27)) (justify left bottom)))
+  (label "WATCHDOG_OK" (at 69.85 116.84 0) (fields_autoplaced yes) (effects (font (size 1.27 1.27)) (justify left bottom)))
+  (label "HEAT_CMD_GPIO" (at 118.11 85.09 0) (fields_autoplaced yes) (effects (font (size 1.27 1.27)) (justify left bottom)))
+  (label "WATCHDOG_OK" (at 118.11 87.63 0) (fields_autoplaced yes) (effects (font (size 1.27 1.27)) (justify left bottom)))
+  (global_label "BROWNOUT_OK" (shape input) (at 118.11 90.17 0) (fields_autoplaced yes) (effects (font (size 1.27 1.27)) (justify left bottom)))
+  (global_label "SAFETY_STATIC_OK" (shape input) (at 118.11 92.71 0) (fields_autoplaced yes) (effects (font (size 1.27 1.27)) (justify left bottom)))
+  (label "NOT_OTA_FAULT" (at 118.11 95.25 0) (fields_autoplaced yes) (effects (font (size 1.27 1.27)) (justify left bottom)))
+  (global_label "RELAY_K1_GATE" (shape output) (at 140.97 87.63 0) (fields_autoplaced yes) (effects (font (size 1.27 1.27)) (justify left bottom)))
+  (global_label "RELAY_K2_GATE" (shape output) (at 140.97 95.25 0) (fields_autoplaced yes) (effects (font (size 1.27 1.27)) (justify left bottom)))
+  (symbol
+    (lib_id "mastertemp_esp32:NetStub_1pin")
+    (at 74.93 82.55 0)
+    (unit 1)
+    (exclude_from_sim yes)
+    (in_bom no)
+    (on_board no)
+    (dnp yes)
+    (property "Reference" "TPI2CSDA" (at 74.93 87.63 0) (effects (font (size 1.27 1.27))))
+    (property "Value" "I2C_SDA_REVIEW_STUB" (at 74.93 90.17 0) (effects (font (size 1.27 1.27))))
+    (property "Footprint" "" (at 74.93 82.55 0) (effects (font (size 1.27 1.27)) (hide yes)))
+    (property "Datasheet" "~" (at 74.93 82.55 0) (effects (font (size 1.27 1.27)) (hide yes)))
+    (property "Description" "Schematic-only review stub until I2C targets and pullups are captured" (at 74.93 82.55 0) (effects (font (size 1.27 1.27)) (hide yes)))
+    (pin "1")
+    (instances (project "mastertemp_esp32" (path "/55f88e14-a963-4749-b9bf-a5d12f0d95cb" (reference "TPI2CSDA") (unit 1))))
+  )
+  (symbol
+    (lib_id "mastertemp_esp32:NetStub_1pin")
+    (at 74.93 85.09 0)
+    (unit 1)
+    (exclude_from_sim yes)
+    (in_bom no)
+    (on_board no)
+    (dnp yes)
+    (property "Reference" "TPI2CSCL" (at 74.93 90.17 0) (effects (font (size 1.27 1.27))))
+    (property "Value" "I2C_SCL_REVIEW_STUB" (at 74.93 92.71 0) (effects (font (size 1.27 1.27))))
+    (property "Footprint" "" (at 74.93 85.09 0) (effects (font (size 1.27 1.27)) (hide yes)))
+    (property "Datasheet" "~" (at 74.93 85.09 0) (effects (font (size 1.27 1.27)) (hide yes)))
+    (property "Description" "Schematic-only review stub until I2C targets and pullups are captured" (at 74.93 85.09 0) (effects (font (size 1.27 1.27)) (hide yes)))
+    (pin "1")
+    (instances (project "mastertemp_esp32" (path "/55f88e14-a963-4749-b9bf-a5d12f0d95cb" (reference "TPI2CSCL") (unit 1))))
   )
   (sheet_instances

Commit message: AI
Parts:
- added R25: I2C_SDA_PULLUP_TBD, Resistor_SMD:R_0805_2012Metric, symbol mastertemp_esp32:Resistor_2pin
- added R26: I2C_SCL_PULLUP_TBD, Resistor_SMD:R_0805_2012Metric, symbol mastertemp_esp32:Resistor_2pin
- added TP4: WATCHDOG_OK, TestPoint_Pad_D2.0mm, symbol mastertemp_esp32:NetStub_1pin
- added U6: MCP23017-E/SS, Package_SO:SSOP-28_5.3x10.2mm_P0.65mm, symbol mastertemp_esp32:MCP23017_SS
- U21: renamed from U9; value RELAY_GATE_LOGIC_TBD -> RELAY_GATE_LOGIC_REVIEW; now not fitted; now left out of the parts list
- U4: value WATCHDOG_SUPERVISOR_TBD -> TPS3823-33DBVR
- U5: value ESP32-WROOM-32E-N16_CANDIDATE -> ESP32-WROOM-32E-N16; footprint RF_Module:ESP32-WROOM-32 -> ESP32-WROOM-32E
Connections:
- net +3V3: now also U4.5 (+3V3), U5.2 (GND), R25.1 (A), R26.1 (A), U6.18 (~{RESET}), U6.9 (VDD); no longer U4.1 (+3V3), U5.1 (+3V3)
- net BROWNOUT_OK: no longer U5.3 (ESP32_EN)
- net GND: now also U5.1 (+3V3), U6.10 (VSS), U6.15 (A0), U6.16 (A1), U6.17 (A2); no longer U5.2 (GND)
- net HEAT_CMD_GPIO: no longer U5.4 (HEAT_CMD_GPIO)
- net I2C_SCL: now also R26.2 (B), U6.12 (SCL); no longer TPI2CSCL.1 (NET), U5.8 (I2C_SCL)
- net I2C_SDA: now also R25.2 (B), U6.13 (SDA); no longer TPI2CSDA.1 (NET), U5.7 (I2C_SDA)
- net NOT_OTA_FAULT: no longer U5.6 (NOT_OTA_FAULT)
- net WATCHDOG_OK: now also U4.1 (WATCHDOG_OK), TP4.1 (NET); no longer U4.4 (WATCHDOG_OK)
- net RELAY_K1_GATE renamed RELAY_K1_GATE_DRIVE
- net RELAY_K2_GATE renamed RELAY_K2_GATE_DRIVE
- net WDI_HEARTBEAT: no longer names the net of U4.3 (WDI)
- net WDI_HEARTBEAT: no longer U5.5 (WDI_HEARTBEAT)
- new net ESP32_EN: U5.3 (ESP32_EN)
- new net IND_OPTO_GPIO: U6.23 (GPA2)
- new net TH_OPTO_GPIO: U6.22 (GPA1)
- new net VAC24_OPTO_GPIO: U6.24 (GPA3)
- new net VAL_OPTO_GPIO: U6.21 (GPA0)
- no-connect marks 0 -> 23
Other:
- moved on the sheet: TPI2CSCL, TPI2CSDA
