File: pcb/mastertemp_esp32/sheets/icm_interface.kicad_sch (KiCad schematic)
At the start: 0 parts

Commit message: Bump
Other:
- note added: "HEAT REQUEST CONTACT PATH: ICM_24VAC_SOURCE -> K1_COM -> K1_NO -> K2_COM -> K2_NO -> TH_HEAT_REQUEST_OUT. K1 and K2 are normally-open relay contacts in series. Loss of board power opens the path."
- note added: "ICM TERMINAL REFERENCE FROM MANUAL FIGURE 24/25: S1/240, S1/120, L1, L2, S2, TH, IND, VAL, GND are on the OEM ignition-control module. This project preserves the OEM ICM and does not replace ignition, blower, HSI, or gas-valve sequencing."
- note added: "J2 OPERATING CONTROL TERMINALS, MANUAL ORDER: 1 VAL_SENSE_MONITOR_ONLY 2 TH_HEAT_REQUEST_OUT 3 IND_SENSE 4 ICM_GND_REF 5 ICM_24VAC_SOURCE 6 FIREMAN_24VAC 7 FIREMAN_SWITCH_RETURN"
- note added: "RELAY COIL GATING: K1 coil enable = HEAT_CMD plus WATCHDOG_OK plus BROWNOUT_OK. K2 coil enable = HEAT_CMD plus SAFETY_STATIC_OK plus NOT_OTA plus NOT_FAULT_LOCKOUT. Every relay-driver gate needs a pulldown so reset/boot/crash keeps heat off."
- note added: "SCHEMATIC PASS 1 - CONTROL BOARD INTERFACE FROM MASTERTEMP 125 REV C FIGURE 24/25"
- note added: "SENSE-ONLY CHANNELS: VAL, IND, TH feedback, and 24VAC presence are isolated AC optocoupler inputs. VAL and GAS are diagnostic monitor inputs only; they must never be sourced or driven by this board."
- note removed: "TODO: J2, dual series NO relays for TH, opto-isolated TH/IND/VAL/24VAC sense, relay feedback."
Changed lines of the file:
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@@
     (comment 1 "TH heat request only. VAL, IND, TH, and 24 VAC are monitor/sense points as defined.")
   )
-  (text "TODO: J2, dual series NO relays for TH, opto-isolated TH/IND/VAL/24VAC sense, relay feedback."
+  (text "SCHEMATIC PASS 1 - CONTROL BOARD INTERFACE FROM MASTERTEMP 125 REV C FIGURE 24/25"
     (at 25.4 25.4 0)
-    (effects (font (size 1.5 1.5)) (justify left bottom))
+    (effects (font (size 1.8 1.8) (bold yes)) (justify left bottom))
   )
   (text "NO GAS VALVE DRIVE OUTPUT ON THIS SHEET."
@@
     (effects (font (size 2.0 2.0) (bold yes)) (justify left bottom))
   )
+  (text "J2 OPERATING CONTROL TERMINALS, MANUAL ORDER:\n1 VAL_SENSE_MONITOR_ONLY\n2 TH_HEAT_REQUEST_OUT\n3 IND_SENSE\n4 ICM_GND_REF\n5 ICM_24VAC_SOURCE\n6 FIREMAN_24VAC\n7 FIREMAN_SWITCH_RETURN"
+    (at 25.4 50.8 0)
+    (effects (font (size 1.35 1.35)) (justify left top))
+  )
+  (text "HEAT REQUEST CONTACT PATH:\nICM_24VAC_SOURCE -> K1_COM -> K1_NO -> K2_COM -> K2_NO -> TH_HEAT_REQUEST_OUT.\nK1 and K2 are normally-open relay contacts in series. Loss of board power opens the path."
+    (at 95.25 50.8 0)
+    (effects (font (size 1.35 1.35)) (justify left top))
+  )
+  (text "RELAY COIL GATING:\nK1 coil enable = HEAT_CMD plus WATCHDOG_OK plus BROWNOUT_OK.\nK2 coil enable = HEAT_CMD plus SAFETY_STATIC_OK plus NOT_OTA plus NOT_FAULT_LOCKOUT.\nEvery relay-driver gate needs a pulldown so reset/boot/crash keeps heat off."
+    (at 95.25 82.55 0)
+    (effects (font (size 1.35 1.35)) (justify left top))
+  )
+  (text "SENSE-ONLY CHANNELS:\nVAL, IND, TH feedback, and 24VAC presence are isolated AC optocoupler inputs.\nVAL and GAS are diagnostic monitor inputs only; they must never be sourced or driven by this board."
+    (at 25.4 101.6 0)
+    (effects (font (size 1.35 1.35)) (justify left top))
+  )
+  (text "ICM TERMINAL REFERENCE FROM MANUAL FIGURE 24/25:\nS1/240, S1/120, L1, L2, S2, TH, IND, VAL, GND are on the OEM ignition-control module.\nThis project preserves the OEM ICM and does not replace ignition, blower, HSI, or gas-valve sequencing."
+    (at 25.4 127.0 0)
+    (effects (font (size 1.35 1.35)) (justify left top))
+  )
   (sheet_instances

Commit message: Make open source.
Parts:
- added D2: K1_FLYBACK_TBD, symbol mastertemp_esp32:Diode_2pin
- added D3: K2_FLYBACK_TBD, symbol mastertemp_esp32:Diode_2pin
- added J2: OPERATING_CONTROL_7P, Connector_Phoenix_MC_HighVoltage:PhoenixContact_MSTBA_2,5_7-G-5,08_1x07_P5.08mm_Horizontal, symbol mastertemp_esp32:OperatingControl_7P
- added K1, K2: G5Q-1A-DC5_CANDIDATE, Relay_THT:Relay_SPST_Omron-G5Q-1A, symbol mastertemp_esp32:RelayNO_5pin
- added Q1: RELAY_K1_LOW_SIDE_TBD, Package_TO_SOT_SMD:SOT-23, symbol mastertemp_esp32:LowSideDriver_3pin
- added Q2: RELAY_K2_LOW_SIDE_TBD, Package_TO_SOT_SMD:SOT-23, symbol mastertemp_esp32:LowSideDriver_3pin
- added TPK1GATE: RELAY_K1_GATE_REVIEW_STUB, symbol mastertemp_esp32:NetStub_1pin
- added TPK2GATE: RELAY_K2_GATE_REVIEW_STUB, symbol mastertemp_esp32:NetStub_1pin
Connections:
- new net +5V_RELAY: D2.2 (K), D3.2 (K), K1.5 (COIL_5V), K2.5 (COIL_5V)
- new net GND: Q1.2 (SOURCE), Q2.2 (SOURCE)
- new net HEAT_CHAIN_K1_K2: K1.3 (NO), K2.2 (COM)
- new net ICM_24VAC_SOURCE: J2.5 (24VAC), K1.2 (COM)
- new net K1_COIL_LOW: D2.1 (A), K1.1 (COIL_LOW), Q1.3 (DRAIN)
- new net K2_COIL_LOW: D3.1 (A), K2.1 (COIL_LOW), Q2.3 (DRAIN)
- new net RELAY_K1_GATE: Q1.1 (GATE), TPK1GATE.1 (NET)
- new net RELAY_K2_GATE: Q2.1 (GATE), TPK2GATE.1 (NET)
- new net TH_HEAT_REQUEST_OUT: J2.2 (TH), K2.3 (NO)
- no-connect marks 0 -> 5
Other:
- note added: "ICM terminal reference from manual Figure 24/25: S1/240, S1/120, L1, L2, S2, TH, IND, VAL, GND. This project preserves the OEM ICM and does not replace ignition, blower, HSI, flame proving, or gas-valve sequencing."
- note added: "ICM_24VAC_SOURCE -> K1_COM -> K1_NO -> K2_COM -> K2_NO -> TH_HEAT_REQUEST_OUT. VAL and GAS are diagnostic monitor inputs only; this board must never source or drive the gas valve."
- note added: "J2 OPERATING CONTROL TERMINALS 1 VAL_SENSE_MONITOR_ONLY 2 TH_HEAT_REQUEST_OUT 3 IND_SENSE 4 ICM_GND_REF 5 ICM_24VAC_SOURCE 6 FIREMAN_24VAC 7 FIREMAN_SWITCH_RETURN"
- note added: "J2 operating-control order is manual-assumed from Rev. C Figure 24: VAL, TH, IND, GND, 24VAC, 24VAC, FS. VAL and IND are sense-only. TH is switched only through K1 and K2 normally-open contacts in series."
- note added: "Relay coil gating remains to be captured with drivers/flyback after supervisor and safety sheets are updated. K1 and K2 coil nets are named here for later connection to low-side MOSFETs and +5V_RELAY."
- note removed: "HEAT REQUEST CONTACT PATH: ICM_24VAC_SOURCE -> K1_COM -> K1_NO -> K2_COM -> K2_NO -> TH_HEAT_REQUEST_OUT. K1 and K2 are normally-open relay contacts in series. Loss of board power opens the path."
- note removed: "ICM TERMINAL REFERENCE FROM MANUAL FIGURE 24/25: S1/240, S1/120, L1, L2, S2, TH, IND, VAL, GND are on the OEM ignition-control module. This project preserves the OEM ICM and does not replace ignition, blower, HSI, or gas-valve sequencing."
- note removed: "J2 OPERATING CONTROL TERMINALS, MANUAL ORDER: 1 VAL_SENSE_MONITOR_ONLY 2 TH_HEAT_REQUEST_OUT 3 IND_SENSE 4 ICM_GND_REF 5 ICM_24VAC_SOURCE 6 FIREMAN_24VAC 7 FIREMAN_SWITCH_RETURN"
- note removed: "RELAY COIL GATING: K1 coil enable = HEAT_CMD plus WATCHDOG_OK plus BROWNOUT_OK. K2 coil enable = HEAT_CMD plus SAFETY_STATIC_OK plus NOT_OTA plus NOT_FAULT_LOCKOUT. Every relay-driver gate needs a pulldown so reset/boot/crash keeps heat off."
- note removed: "SENSE-ONLY CHANNELS: VAL, IND, TH feedback, and 24VAC presence are isolated AC optocoupler inputs. VAL and GAS are diagnostic monitor inputs only; they must never be sourced or driven by this board."

Commit message: AI
Parts:
- added R10: K1_GATE_PULLDOWN_TBD, Resistor_SMD:R_0805_2012Metric, symbol mastertemp_esp32:Resistor_2pin
- added R11: K2_GATE_PULLDOWN_TBD, Resistor_SMD:R_0805_2012Metric, symbol mastertemp_esp32:Resistor_2pin
- added R12: VAL_OPTO_PULLUP_TBD, Resistor_SMD:R_0805_2012Metric, symbol mastertemp_esp32:Resistor_2pin
- added R13: TH_OPTO_LIMIT_A_TBD, Resistor_SMD:R_0805_2012Metric, symbol mastertemp_esp32:Resistor_2pin
- added R14: TH_OPTO_LIMIT_B_TBD, Resistor_SMD:R_0805_2012Metric, symbol mastertemp_esp32:Resistor_2pin
- added R15: TH_OPTO_PULLUP_TBD, Resistor_SMD:R_0805_2012Metric, symbol mastertemp_esp32:Resistor_2pin
- added R16: IND_OPTO_LIMIT_A_TBD, Resistor_SMD:R_0805_2012Metric, symbol mastertemp_esp32:Resistor_2pin
- added R17: IND_OPTO_LIMIT_B_TBD, Resistor_SMD:R_0805_2012Metric, symbol mastertemp_esp32:Resistor_2pin
- added R18: IND_OPTO_PULLUP_TBD, Resistor_SMD:R_0805_2012Metric, symbol mastertemp_esp32:Resistor_2pin
- added R19: VAC24_OPTO_LIMIT_A_TBD, Resistor_SMD:R_0805_2012Metric, symbol mastertemp_esp32:Resistor_2pin
- added R20: VAC24_OPTO_LIMIT_B_TBD, Resistor_SMD:R_0805_2012Metric, symbol mastertemp_esp32:Resistor_2pin
- added R21: VAC24_OPTO_PULLUP_TBD, Resistor_SMD:R_0805_2012Metric, symbol mastertemp_esp32:Resistor_2pin
- added R22: K1_GATE_SERIES_TBD, Resistor_SMD:R_0805_2012Metric, symbol mastertemp_esp32:Resistor_2pin
- added R23: K2_GATE_SERIES_TBD, Resistor_SMD:R_0805_2012Metric, symbol mastertemp_esp32:Resistor_2pin
- added R8: VAL_OPTO_LIMIT_A_TBD, Resistor_SMD:R_0805_2012Metric, symbol mastertemp_esp32:Resistor_2pin
- added R9: VAL_OPTO_LIMIT_B_TBD, Resistor_SMD:R_0805_2012Metric, symbol mastertemp_esp32:Resistor_2pin
- added TP6: K1_COIL, TestPoint_Pad_D2.0mm, symbol mastertemp_esp32:NetStub_1pin
- added TP7: K2_COIL, TestPoint_Pad_D2.0mm, symbol mastertemp_esp32:NetStub_1pin
- added TP8: TH_FEEDBACK, TestPoint_Pad_D2.0mm, symbol mastertemp_esp32:NetStub_1pin
- added TP9: VAL_SENSE, TestPoint_Pad_D2.0mm, symbol mastertemp_esp32:NetStub_1pin
- added U10: H11AA1M_IND, Package_DIP:DIP-6_W7.62mm, symbol mastertemp_esp32:H11AA1M
- added U11: H11AA1M_VAL, Package_DIP:DIP-6_W7.62mm, symbol mastertemp_esp32:H11AA1M
- added U12: H11AA1M_24VAC, Package_DIP:DIP-6_W7.62mm, symbol mastertemp_esp32:H11AA1M
- added U9: H11AA1M_TH, Package_DIP:DIP-6_W7.62mm, symbol mastertemp_esp32:H11AA1M
- D2, D3: footprint (none) -> Diode_SMD:D_SOD-123
- J2: value OPERATING_CONTROL_7P -> OPERATING_CONTROL; footprint Connector_Phoenix_MC_HighVoltage:PhoenixContact_MSTBA_2,5_7-G-5,08_1x07_P5.08mm_Horizontal -> Connector_Phoenix_MSTB:PhoenixContact_MSTBA_2,5_7-G-5,08_1x07_P5.08mm_Horizontal
- K1, K2: value G5Q-1A-DC5_CANDIDATE -> G5Q-1A-DC5
- Q1: value RELAY_K1_LOW_SIDE_TBD -> AO3400A
- Q2: value RELAY_K2_LOW_SIDE_TBD -> AO3400A
Connections:
- net +5V_RELAY: now also D2.1 (A), D3.1 (A); no longer D2.2 (K), D3.2 (K)
- net GND: now also R10.2 (B), R11.2 (B), U10.4 (EMITTER), U11.4 (EMITTER), U12.4 (EMITTER), U9.4 (EMITTER)
- net ICM_24VAC_SOURCE: now also R19.1 (A)
- net K1_COIL_LOW: now also D2.2 (K), TP6.1 (NET); no longer D2.1 (A)
- net K2_COIL_LOW: now also D3.2 (K), TP7.1 (NET); no longer D3.1 (A)
- net RELAY_K1_GATE: now also R10.1 (A), R22.2 (B)
- net RELAY_K2_GATE: now also R11.1 (A), R23.2 (B)
- net TH_HEAT_REQUEST_OUT: now also R13.1 (A)
- net VAL_SENSE_AC: now reaches J2.1 (VAL)
- net VAL_SENSE_AC: now also R8.1 (A), TP9.1 (NET)
- net IND_SENSE_AC: now reaches J2.3 (IND)
- net IND_SENSE_AC: now also R16.1 (A)
- net ICM_GND_REF: now reaches J2.4 (GND)
- net ICM_GND_REF: now also U10.2 (AC_IN_2), U11.2 (AC_IN_2), U12.2 (AC_IN_2), U9.2 (AC_IN_2)
- net FIREMAN_24VAC: now reaches J2.6 (FS_24VAC)
- net FIREMAN_SWITCH_RETURN: now reaches J2.7 (FS_RETURN)
- new net +3V3: R12.2 (B), R15.2 (B), R18.2 (B), R21.2 (B)
- new net IND_OPTO_GPIO: R18.1 (A), U10.5 (COLLECTOR)
- new net IND_OPTO_INPUT: R17.2 (B), U10.1 (AC_IN_1)
- new net IND_OPTO_LIMIT_A: R16.2 (B), R17.1 (A)
- new net RELAY_K1_GATE_DRIVE: R22.1 (A)
- new net RELAY_K2_GATE_DRIVE: R23.1 (A)
- new net TH_FEEDBACK: TP8.1 (NET)
- new net TH_OPTO_GPIO: R15.1 (A), U9.5 (COLLECTOR)
- new net TH_OPTO_INPUT: R14.2 (B), U9.1 (AC_IN_1)
- new net TH_OPTO_LIMIT_A: R13.2 (B), R14.1 (A)
- new net VAC24_OPTO_GPIO: R21.1 (A), U12.5 (COLLECTOR)
- new net VAC24_OPTO_INPUT: R20.2 (B), U12.1 (AC_IN_1)
- new net VAC24_OPTO_LIMIT_A: R19.2 (B), R20.1 (A)
- new net VAL_OPTO_GPIO: R12.1 (A), U11.5 (COLLECTOR)
- new net VAL_OPTO_INPUT: R9.2 (B), U11.1 (AC_IN_1)
- new net VAL_OPTO_LIMIT_A: R8.2 (B), R9.1 (A)
- no-connect marks 5 -> 4
