File: pcb/mastertemp_esp32/sheets/power_24vac.kicad_sch (KiCad schematic)
At the start: 0 parts

Commit message: Make open source.
Parts:
- added D1: BRIDGE_RECTIFIER_TBD, symbol mastertemp_esp32:Bridge_4pin
- added F1: 0.5A_PTC_OR_FUSE_TBD, symbol mastertemp_esp32:Fuse_2pin
- added J1: POWER_24VAC_3P, Connector_Phoenix_MC_HighVoltage:PhoenixContact_MSTBA_2,5_3-G-5,08_1x03_P5.08mm_Horizontal, symbol mastertemp_esp32:PowerEntry_3P
- added TPBROWN: BROWNOUT_OK_REVIEW_STUB, symbol mastertemp_esp32:NetStub_1pin
- added TPP3GOOD: +3V3_PGOOD_REVIEW_STUB, symbol mastertemp_esp32:NetStub_1pin
- added TPP3V3: +3V3_REVIEW_STUB, symbol mastertemp_esp32:NetStub_1pin
- added TPP5V: +5V_REVIEW_STUB, symbol mastertemp_esp32:NetStub_1pin
- added TPPGOOD: +5V_PGOOD_REVIEW_STUB, symbol mastertemp_esp32:NetStub_1pin
- added TPSHIELD: CHASSIS_SHIELD_REVIEW_STUB, symbol mastertemp_esp32:NetStub_1pin
- added U1: LM5164_100V_BUCK_5V, Package_DFN_QFN:Texas_S-PVSON-N10, symbol mastertemp_esp32:PowerBuck_5pin
- added U2: 3V3_BUCK_OR_REGULATOR_TBD, Package_TO_SOT_SMD:TSOT-23-6, symbol mastertemp_esp32:PowerBuck_5pin
- added U3: 3V3_RESET_SUPERVISOR_TBD, Package_TO_SOT_SMD:SOT-23, symbol mastertemp_esp32:Supervisor_3pin
Connections:
- new net +3V3: TPP3V3.1 (NET), U2.4 (VOUT), U3.3 (VDD)
- new net +3V3_PGOOD: TPP3GOOD.1 (NET), U2.5 (PGOOD)
- new net +5V: TPP5V.1 (NET), U1.4 (VOUT), U2.1 (VIN), U2.3 (EN)
- new net +5V_PGOOD: TPPGOOD.1 (NET), U1.5 (PGOOD)
- new net BROWNOUT_OK: TPBROWN.1 (NET), U3.2 (~{RESET})
- new net CHASSIS_SHIELD: J1.3 (SHIELD), TPSHIELD.1 (NET)
- new net PGND_RAW: D1.4 (-), U1.2 (GND), U2.2 (GND), U3.1 (GND)
- new net VAC24_A: F1.2 (B), J1.1 (VAC24_A)
- new net VAC24_A_FUSED: D1.1 (AC1), F1.1 (A)
- new net VAC24_B: D1.2 (AC2), J1.2 (VAC24_B)
- new net VRAW: D1.3 (+), U1.1 (VIN), U1.3 (EN)
Other:
- note added: "Final fuse, MOV/TVS, buck compensation, inductor, diode, capacitor, and divider values remain open until transformer measurements are recorded."
- note added: "J1 brings in the heater control transformer secondary only. No line voltage is permitted on this PCB."
- note added: "Power-tree net names captured on this pass: VAC24_A/B -> VAC24_A_FUSED -> VRAW/PGND_RAW -> +5V -> +3V3 -> BROWNOUT_OK. Detailed wires and support passives are the next schematic increment."
- note added: "Protection/capture intent: fuse or PTC in VAC24_A, MOV/TVS surge clamp, bridge rectifier, VRAW bulk rated for unloaded transformer margin."
- note added: "Regulator intent: U1 100 V buck generates +5V; U2 generates +3V3; U3 asserts BROWNOUT_OK/ESP32_EN only after +3V3 is valid."
- note added: "SCHEMATIC PASS 1 - MANUAL-ASSUMED 24 VAC POWER TREE"
- note removed: "TODO: J1, fuse/PTC, MOV/TVS, bridge, VRAW bulk, 5 V buck, 3.3 V regulator, brownout supervisor."

Commit message: AI
Parts:
- added C1: 470uF_63V, Capacitor_THT:CP_Radial_D10.0mm_P5.00mm, symbol mastertemp_esp32:Capacitor_2pin
- added C4: 2.2uF_100V_VRAW_IN_TBD, Capacitor_SMD:C_1210_3225Metric, symbol mastertemp_esp32:Capacitor_2pin
- added C5: 2.2nF_50V_BST_5V, Capacitor_SMD:C_0603_1608Metric, symbol mastertemp_esp32:Capacitor_2pin
- added C6: 100nF_BST_3V3, Capacitor_SMD:C_0603_1608Metric, symbol mastertemp_esp32:Capacitor_2pin
- added C7: 10uF_50V_3V3_IN_TBD, Capacitor_SMD:C_1210_3225Metric, symbol mastertemp_esp32:Capacitor_2pin
- added C8: 22uF_10V_3V3_OUT_TBD, Capacitor_SMD:C_0805_2012Metric, symbol mastertemp_esp32:Capacitor_2pin
- added L1: 68uH, Inductor_SMD:L_12x12mm_H8mm, symbol mastertemp_esp32:Inductor_2pin
- added L2: 2.2uH, Inductor_SMD:L_Vishay_IFSC-1515AH_4x4x1.8mm, symbol mastertemp_esp32:Inductor_2pin
- added MOV1: V47ZA1P, Varistor:RV_Disc_D7mm_W3.9mm_P5mm, symbol mastertemp_esp32:Resistor_2pin
- added R5: RFB5V_TOP_TBD, Resistor_SMD:R_0805_2012Metric, symbol mastertemp_esp32:Resistor_2pin
- added R6: RFB5V_BOT_TBD, Resistor_SMD:R_0805_2012Metric, symbol mastertemp_esp32:Resistor_2pin
- added R7: RON5V_TBD, Resistor_SMD:R_0805_2012Metric, symbol mastertemp_esp32:Resistor_2pin
- added TP1: VRAW, TestPoint_Pad_D2.0mm, symbol mastertemp_esp32:NetStub_1pin
- added TP2: +5V, TestPoint_Pad_D2.0mm, symbol mastertemp_esp32:NetStub_1pin
- added TP3: +3V3, TestPoint_Pad_D2.0mm, symbol mastertemp_esp32:NetStub_1pin
- added TVS1: SMBJ51CA, Diode_SMD:D_SMB, symbol mastertemp_esp32:Diode_2pin
- added U8: NXE1S0505MC-R7, Converter_DCDC:Converter_DCDC_Murata_NXExSxxxxMC_SMD, symbol mastertemp_esp32:Uncommitted_NXE5
- D1: value BRIDGE_RECTIFIER_TBD -> MB10S; footprint (none) -> Diode_SMD:Diode_Bridge_Vishay_MBLS
- F1: value 0.5A_PTC_OR_FUSE_TBD -> 0.5A_FUSE; footprint (none) -> Fuse:Fuse_1206_3216Metric
- J1: value POWER_24VAC_3P -> 24VAC_IN; footprint Connector_Phoenix_MC_HighVoltage:PhoenixContact_MSTBA_2,5_3-G-5,08_1x03_P5.08mm_Horizontal -> Connector_Phoenix_MSTB:PhoenixContact_MSTBA_2,5_3-G-5,08_1x03_P5.08mm_Horizontal
- U1: value LM5164_100V_BUCK_5V -> LM5164DDAR; footprint Package_DFN_QFN:Texas_S-PVSON-N10 -> Package_SO:TI_SO-PowerPAD-8; symbol mastertemp_esp32:PowerBuck_5pin -> mastertemp_esp32:LM5164_DDA8
- U2: value 3V3_BUCK_OR_REGULATOR_TBD -> AP63203WU-7; symbol mastertemp_esp32:PowerBuck_5pin -> mastertemp_esp32:AP63203_TSOT26
- U3: value 3V3_RESET_SUPERVISOR_TBD -> TPS3839G33DBZR; footprint Package_TO_SOT_SMD:SOT-23 -> Package_TO_SOT_SMD:SOT-23-3
Connections:
- net +3V3: now also U2.1 (FB), C8.1 (A), L2.2 (B), TP3.1 (NET); no longer TPP3V3.1 (NET), U2.4 (VOUT)
- net +5V: now also U2.2 (EN), C7.1 (A), L1.2 (B), R5.1 (A), TP2.1 (NET), U8.3 (PAD3); no longer TPP5V.1 (NET), U1.4 (VOUT), U2.1 (VIN)
- net +5V_PGOOD: now also TPP5V.1 (NET), U1.6 (PGOOD); no longer TPPGOOD.1 (NET), U1.5 (PGOOD)
- net BROWNOUT_OK: now also U3.1 (~{RESET}); no longer U3.2 (~{RESET})
- net PGND_RAW: now also U1.1 (GND), U1.9 (EP), C1.2 (B), C4.2 (B), R6.2 (B), R7.2 (B); no longer U1.2 (GND), U2.2 (GND), U3.1 (GND)
- net VAC24_A_FUSED: now also MOV1.1 (A), TVS1.1 (A)
- net VAC24_B: now also MOV1.2 (B), TVS1.2 (K)
- net VRAW: now also U1.2 (VIN), C1.1 (A), C4.1 (A), TP1.1 (NET); no longer U1.1 (VIN)
- net +3V3_PGOOD renamed BST_3V3
- net BST_3V3: now also U2.6 (BST), C6.1 (A); no longer U2.5 (PGOOD)
- new net BST_5V: C5.1 (A), U1.7 (BST)
- new net COMMON_LINE: U8.7 (PAD7)
- new net FB_5V_TBD: R5.2 (B), R6.1 (A), U1.5 (FB)
- new net GND: C7.2 (B), C8.2 (B), U2.5 (GND), U3.2 (GND), U8.1 (PAD1)
- new net ISO_REMOTE_5V: U8.8 (PAD8)
- new net RON_5V_TBD: R7.1 (A), U1.4 (RON)
- new net SW_3V3: C6.2 (B), L2.1 (A), TPP3V3.1 (NET), U2.4 (SW)
- new net SW_5V: C5.2 (B), L1.1 (A), TPPGOOD.1 (NET), U1.8 (SW)
- no-connect marks 0 -> 1
Other:
- note added: "Power-tree nets and draft support parts captured on this pass: VAC24_A/B -> VAC24_A_FUSED -> VRAW/PGND_RAW -> SW_5V/+5V -> +3V3 -> BROWNOUT_OK. Final fuse, clamp, buck-compensation, inductor, diode, capacitor, and divider values remain open until measurements."
- note removed: "Power-tree net names captured on this pass: VAC24_A/B -> VAC24_A_FUSED -> VRAW/PGND_RAW -> +5V -> +3V3 -> BROWNOUT_OK. Detailed wires and support passives are the next schematic increment."
