File: pcb/mastertemp_esp32/sheets/thermistor_sfs.kicad_sch (KiCad schematic)
At the start: 0 parts

Commit message: AI Gen
Parts:
- added J4: THERMISTOR_2P, TerminalBlock_Phoenix:PhoenixContact_MSTBA_2,5_2-G-5,08_1x02_P5.08mm_Horizontal, symbol mastertemp_esp32:SensorConnector_2P
- added TP3V3ADC: +3V3_ADC_REVIEW_STUB, symbol mastertemp_esp32:NetStub_1pin
- added TPADC3: ADC_AIN3_SPARE_REVIEW_STUB, symbol mastertemp_esp32:NetStub_1pin
- added TPADCA: ADS1115_ALERT_REVIEW_STUB, symbol mastertemp_esp32:NetStub_1pin
- added TPADCADDR: ADS1115_ADDR_REVIEW_STUB, symbol mastertemp_esp32:NetStub_1pin
- added TPGNDADC: ADC_GND_REVIEW_STUB, symbol mastertemp_esp32:NetStub_1pin
- added TPI2CSCL2: I2C_SCL_REVIEW_STUB, symbol mastertemp_esp32:NetStub_1pin
- added TPI2CSDA2: I2C_SDA_REVIEW_STUB, symbol mastertemp_esp32:NetStub_1pin
- added TPSFSHREF: SFS_HIGH_REF_TBD, symbol mastertemp_esp32:NetStub_1pin
- added TPSFSLREF: SFS_LOW_REF_TBD, symbol mastertemp_esp32:NetStub_1pin
- added TPSFSRET: SFS_RETURN_OR_REF_REVIEW_STUB, symbol mastertemp_esp32:NetStub_1pin
- added TPSFSWGND: SFS_WINDOW_GND_REVIEW_STUB, symbol mastertemp_esp32:NetStub_1pin
- added TPTHHREF: THERM_HIGH_REF_TBD, symbol mastertemp_esp32:NetStub_1pin
- added TPTHLREF: THERM_LOW_REF_TBD, symbol mastertemp_esp32:NetStub_1pin
- added TPTHWGND: THERM_WINDOW_GND_REVIEW_STUB, symbol mastertemp_esp32:NetStub_1pin
- added TPVRAWADC: VRAW_MONITOR_REVIEW_STUB, symbol mastertemp_esp32:NetStub_1pin
- added U14: THERMISTOR_AFE_TBD, symbol mastertemp_esp32:SensorAFE_6pin
- added U16: THERM_WINDOW_TLV6700_TBD, Package_TO_SOT_SMD:SOT-23-6, symbol mastertemp_esp32:WindowComparator_5pin
- added U17: SFS_WINDOW_TLV6700_TBD, Package_TO_SOT_SMD:SOT-23-6, symbol mastertemp_esp32:WindowComparator_5pin
- added U18: SFS_AFE_BUFFER_TBD, Package_TO_SOT_SMD:SOT-23-5, symbol mastertemp_esp32:SensorAFE_6pin
- added U7: ADS1115IDGSR_CANDIDATE, Package_SO:VSSOP-10_3x3mm_P0.5mm, symbol mastertemp_esp32:ADS1115_Block
Connections:
- new net +3V3: TP3V3ADC.1 (NET), U7.5 (+3V3)
- new net +3V3_ADC: U14.3 (+3V3_ADC), U18.3 (+3V3_ADC)
- new net ADC_AIN3_SPARE_REVIEW: TPADC3.1 (NET), U7.4 (AIN3_SPARE)
- new net ADS1115_ADDR_REVIEW: TPADCADDR.1 (NET), U7.10 (ADDR)
- new net ADS1115_ALERT_REVIEW: TPADCA.1 (NET), U7.9 (ALERT)
- new net AGND: U14.4 (AGND), U18.4 (AGND)
- new net GND: TPGNDADC.1 (NET), TPSFSWGND.1 (NET), TPTHWGND.1 (NET), U16.5 (PWR_GND), U17.5 (PWR_GND), U7.6 (GND)
- new net I2C_SCL: TPI2CSCL2.1 (NET), U7.8 (I2C_SCL)
- new net I2C_SDA: TPI2CSDA2.1 (NET), U7.7 (I2C_SDA)
- new net SFS_ADC_AIN1: U18.5 (ADC_OUT), U7.2 (AIN1_SFS)
- new net SFS_FIELD_INPUT: U18.1 (SENSOR_A)
- new net SFS_HIGH_REF_TBD: TPSFSHREF.1 (NET), U17.3 (HIGH_REF)
- new net SFS_LOW_REF_TBD: TPSFSLREF.1 (NET), U17.2 (LOW_REF)
- new net SFS_RANGE_OK: U17.4 (RANGE_OK)
- new net SFS_RETURN_OR_REF: TPSFSRET.1 (NET), U18.2 (SENSOR_B)
- new net SFS_WINDOW_SENSE: U17.1 (SENSE), U18.6 (WINDOW_SENSE)
- new net THERMISTOR_A: J4.1 (A), U14.1 (SENSOR_A)
- new net THERMISTOR_B: J4.2 (B), U14.2 (SENSOR_B)
- new net THERMISTOR_RANGE_OK: U16.4 (RANGE_OK)
- new net THERM_ADC_AIN0: U14.5 (ADC_OUT), U7.1 (AIN0_THERM)
- new net THERM_HIGH_REF_TBD: TPTHHREF.1 (NET), U16.3 (HIGH_REF)
- new net THERM_LOW_REF_TBD: TPTHLREF.1 (NET), U16.2 (LOW_REF)
- new net THERM_WINDOW_SENSE: U14.6 (WINDOW_SENSE), U16.1 (SENSE)
- new net VRAW_MONITOR_REVIEW: TPVRAWADC.1 (NET), U7.3 (AIN2_VRAW)
Other:
- note added: "ADS1115 allocation: AIN0 = water thermistor divider AIN1 = stack flue sensor measurement AIN2 = VRAW/rail monitor review stub AIN3 = spare/review stub I2C pullups and address strap values remain TBD."
- note added: "SCHEMATIC PASS 1 - SENSOR MEASUREMENT AND HARDWARE RANGE GATES"
- note added: "SFS front end is intentionally abstract: SFS electrical type/range is TBD. Use high-impedance excitation or buffer only after measuring the installed harness. SFS_RANGE_OK must drop on open, short, overtemperature/fault, or out-of-window behavior without firmware help."
- note added: "Thermistor front end follows preliminary design intent: protected divider, 10 k 0.1 percent pull-up target, ADC filter, and independent hardware window comparator. Final curve, thresholds, resistor values, pull-up rail, and fault thresholds require field verification against the installed sensor."
- note removed: "TODO: thermistor divider, SFS excitation/buffer, ADS1115, hardware window comparators, ESD protection."

Commit message: AI
Parts:
- added C10: SFS_ADC_FILTER_TBD, Capacitor_SMD:C_0805_2012Metric, symbol mastertemp_esp32:Capacitor_2pin
- added C11: VRAW_MON_FILTER_TBD, Capacitor_SMD:C_0805_2012Metric, symbol mastertemp_esp32:Capacitor_2pin
- added C9: THERM_ADC_FILTER_TBD, Capacitor_SMD:C_0805_2012Metric, symbol mastertemp_esp32:Capacitor_2pin
- added R24: THERM_PULLUP_TBD, Resistor_SMD:R_0805_2012Metric, symbol mastertemp_esp32:Resistor_2pin
- added R27: SFS_INPUT_SERIES_TBD, Resistor_SMD:R_0805_2012Metric, symbol mastertemp_esp32:Resistor_2pin
- added R28: VRAW_MON_TOP_TBD, Resistor_SMD:R_0805_2012Metric, symbol mastertemp_esp32:Resistor_2pin
- added R29: VRAW_MON_BOT_TBD, Resistor_SMD:R_0805_2012Metric, symbol mastertemp_esp32:Resistor_2pin
- added R30: THERM_RANGE_OK_PULLUP_TBD, Resistor_SMD:R_0805_2012Metric, symbol mastertemp_esp32:Resistor_2pin
- added R31: SFS_RANGE_OK_PULLUP_TBD, Resistor_SMD:R_0805_2012Metric, symbol mastertemp_esp32:Resistor_2pin
- added R32: THERM_LOW_REF_TOP_TBD, Resistor_SMD:R_0805_2012Metric, symbol mastertemp_esp32:Resistor_2pin
- added R33: THERM_LOW_REF_BOT_TBD, Resistor_SMD:R_0805_2012Metric, symbol mastertemp_esp32:Resistor_2pin
- added R34: THERM_HIGH_REF_TOP_TBD, Resistor_SMD:R_0805_2012Metric, symbol mastertemp_esp32:Resistor_2pin
- added R35: THERM_HIGH_REF_BOT_TBD, Resistor_SMD:R_0805_2012Metric, symbol mastertemp_esp32:Resistor_2pin
- added R36: SFS_LOW_REF_TOP_TBD, Resistor_SMD:R_0805_2012Metric, symbol mastertemp_esp32:Resistor_2pin
- added R37: SFS_LOW_REF_BOT_TBD, Resistor_SMD:R_0805_2012Metric, symbol mastertemp_esp32:Resistor_2pin
- added R38: SFS_HIGH_REF_TOP_TBD, Resistor_SMD:R_0805_2012Metric, symbol mastertemp_esp32:Resistor_2pin
- added R39: SFS_HIGH_REF_BOT_TBD, Resistor_SMD:R_0805_2012Metric, symbol mastertemp_esp32:Resistor_2pin
- J4: value THERMISTOR_2P -> THERMISTOR; footprint TerminalBlock_Phoenix:PhoenixContact_MSTBA_2,5_2-G-5,08_1x02_P5.08mm_Horizontal -> Connector_Phoenix_MSTB:PhoenixContact_MSTBA_2,5_2-G-5,08_1x02_P5.08mm_Horizontal
- U14: footprint (none) -> Package_TO_SOT_SMD:SOT-23-6
- U16: value THERM_WINDOW_TLV6700_TBD -> TLV6700DDCR_THERM
- U17: value SFS_WINDOW_TLV6700_TBD -> TLV6700DDCR_SFS
- U18: value SFS_AFE_BUFFER_TBD -> OPA333AIDBVR; symbol mastertemp_esp32:SensorAFE_6pin -> mastertemp_esp32:SFSBuffer_5pin
- U7: value ADS1115IDGSR_CANDIDATE -> ADS1115IDGSR
Connections:
- net ADC_AIN3_SPARE_REVIEW is gone; now on net I2C_SCL: TPADC3.1 (NET), U7.4 (AIN3_SPARE)
- net ADS1115_ADDR_REVIEW is gone; now on net +3V3: TPADCADDR.1 (NET), U7.10 (ADDR)
- net VRAW_MONITOR_REVIEW is gone; now on net I2C_SDA: TPVRAWADC.1 (NET), U7.3 (AIN2_VRAW)
- net +3V3: now also R30.1 (A), R31.1 (A); no longer TP3V3ADC.1 (NET), U7.5 (+3V3)
- net +3V3_ADC: now also R24.1 (A), R32.1 (A), R34.1 (A), R36.1 (A), R38.1 (A)
- net AGND: now also C10.2 (B), C11.2 (B), C9.2 (B), R29.2 (B), R33.2 (B), R35.2 (B), R37.2 (B), R39.2 (B)
- net GND: now also TP3V3ADC.1 (NET), U7.5 (+3V3); no longer TPGNDADC.1 (NET), U7.6 (GND)
- net I2C_SCL: no longer TPI2CSCL2.1 (NET), U7.8 (I2C_SCL)
- net I2C_SDA: no longer TPI2CSDA2.1 (NET), U7.7 (I2C_SDA)
- net SFS_FIELD_INPUT: now also R27.2 (B)
- net SFS_HIGH_REF_TBD: now also R38.2 (B), R39.1 (A)
- net SFS_LOW_REF_TBD: now also R36.2 (B), R37.1 (A)
- net SFS_RANGE_OK: now also R31.2 (B)
- net SFS_WINDOW_SENSE: no longer U18.6 (WINDOW_SENSE)
- net THERMISTOR_RANGE_OK: now also R30.2 (B)
- net THERM_HIGH_REF_TBD: now also R34.2 (B), R35.1 (A)
- net THERM_LOW_REF_TBD: now also R32.2 (B), R33.1 (A)
- net ADS1115_ALERT_REVIEW renamed VAL_SENSE_ADC
- net SFS_ADC_AIN1: no longer names the net of U7.2 (AIN1_SFS)
- net SFS_ADC_AIN1: no longer U18.5 (ADC_OUT)
- net THERM_ADC_AIN0: no longer names the net of U7.1 (AIN0_THERM)
- net THERM_ADC_AIN0: no longer U14.5 (ADC_OUT)
- new net SFS_ADC: C10.1 (A), TPI2CSDA2.1 (NET), U18.5 (SFS_ADC), U7.7 (I2C_SDA)
- new net SFS_INPUT: R27.1 (A)
- new net THERMISTOR_ADC: C9.1 (A), R24.2 (B), TPGNDADC.1 (NET), U14.5 (ADC_OUT), U7.6 (GND)
- new net VRAW: R28.1 (A)
- new net VRAW_MONITOR_ADC: C11.1 (A), R28.2 (B), R29.1 (A), TPI2CSCL2.1 (NET), U7.8 (I2C_SCL)
- no-connect marks 0 -> 2
