File: pcb/mastertemp_esp32/sheets/ui_remote.kicad_sch (KiCad schematic)
At the start: 0 parts

Commit message: Bump
Other:
- note added: "FIRMWARE/UI POLICY: Local keypad behavior, if retained, must not bypass hardware lockouts. MQTT/Home Assistant commands remain advisory and cannot override any safety fault."
- note added: "J5 EXTERNAL CONTROL INTERFACE FROM MANUAL FIGURE 24: 1 SPA_LINE 2 COMMON_LINE 3 POOL_LINE Use isolated dry-contact sensing. If Pool and Spa are both asserted, fault and keep heat off."
- note added: "J6 OEM MEMBRANE CONNECTOR: Reference only for compatibility with the original control board layout. No replacement keypad electronics are designed in this project."
- note added: "KEYPAD / MEMBRANE PAD / DISPLAY / BUZZER / STATUS LED DESIGN IS OUT OF SCOPE. This sheet only captures the control-board external control interface needed to request Pool, Spa, or Off behavior."
- note added: "SCHEMATIC PASS 1 - EXTERNAL CONTROL ONLY"
- note removed: "TODO: Pool/Common/Spa dry-contact inputs, local buttons, OLED/I2C, buzzer, status LEDs."
- title: Remote Controls, Local UI, Display, Status Outputs -> External Control Interface - Keypad Out of Scope
Changed lines of the file:
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@@
   (paper "A3")
   (title_block
-    (title "Remote Controls, Local UI, Display, Status Outputs")
+    (title "External Control Interface - Keypad Out of Scope")
     (date "2026-05-31")
     (rev "scaffold-0")
     (company "Preliminary - not certified")
-    (comment 1 "Pool/Common/Spa remote inputs are dry-contact sensing only.")
+    (comment 1 "Pool/Common/Spa remote inputs are dry-contact sensing only. No keypad/display design.")
   )
-  (text "TODO: Pool/Common/Spa dry-contact inputs, local buttons, OLED/I2C, buzzer, status LEDs."
+  (text "SCHEMATIC PASS 1 - EXTERNAL CONTROL ONLY"
     (at 25.4 25.4 0)
-    (effects (font (size 1.5 1.5)) (justify left bottom))
+    (effects (font (size 1.8 1.8) (bold yes)) (justify left bottom))
+  )
+  (text "KEYPAD / MEMBRANE PAD / DISPLAY / BUZZER / STATUS LED DESIGN IS OUT OF SCOPE.\nThis sheet only captures the control-board external control interface needed to request Pool, Spa, or Off behavior."
+    (at 25.4 38.1 0)
+    (effects (font (size 1.5 1.5) (bold yes)) (justify left top))
+  )
+  (text "J5 EXTERNAL CONTROL INTERFACE FROM MANUAL FIGURE 24:\n1 SPA_LINE\n2 COMMON_LINE\n3 POOL_LINE\nUse isolated dry-contact sensing. If Pool and Spa are both asserted, fault and keep heat off."
+    (at 25.4 69.85 0)
+    (effects (font (size 1.35 1.35)) (justify left top))
+  )
+  (text "J6 OEM MEMBRANE CONNECTOR:\nReference only for compatibility with the original control board layout.\nNo replacement keypad electronics are designed in this project."
+    (at 25.4 101.6 0)
+    (effects (font (size 1.35 1.35)) (justify left top))
+  )
+  (text "FIRMWARE/UI POLICY:\nLocal keypad behavior, if retained, must not bypass hardware lockouts.\nMQTT/Home Assistant commands remain advisory and cannot override any safety fault."
+    (at 25.4 127.0 0)
+    (effects (font (size 1.35 1.35)) (justify left top))
   )
   (sheet_instances

Commit message: AI
Parts:
- added C2, C3: 100nF_REMOTE_FILTER_TBD, Capacitor_SMD:C_0805_2012Metric, symbol mastertemp_esp32:Capacitor_2pin
- added J5: EXT_CONTROL, Connector_Phoenix_MSTB:PhoenixContact_MSTBA_2,5_3-G-5,08_1x03_P5.08mm_Horizontal, symbol mastertemp_esp32:ExternalControl_3P
- added J6: MEMBRANE_REF, Connector_Phoenix_MSTB:PhoenixContact_MSTBVA_2,5_9-G-5,08_1x09_P5.08mm_Vertical, symbol mastertemp_esp32:MembraneReference_9P
- added R1, R2: 2.2k_REMOTE_WET_TBD, Resistor_SMD:R_0805_2012Metric, symbol mastertemp_esp32:Resistor_2pin
- added R3, R4: 10k_REMOTE_PULLUP, Resistor_SMD:R_0805_2012Metric, symbol mastertemp_esp32:Resistor_2pin
- added U19: LTV-817S_SPA_CANDIDATE, Package_DIP:DIP-4_W7.62mm, symbol mastertemp_esp32:Optocoupler_4pin
- added U20: LTV-817S_POOL_CANDIDATE, Package_DIP:DIP-4_W7.62mm, symbol mastertemp_esp32:Optocoupler_4pin
Connections:
- new net +3V3: R3.1 (A), R4.1 (A)
- new net COMMON_LINE: J5.2 (COMMON)
- new net GND: C2.2 (B), C3.2 (B), U19.3 (EMITTER), U20.3 (EMITTER)
- new net ISO_REMOTE_5V: R1.1 (A), R2.1 (A)
- new net POOL_LED_A: R2.2 (B), U20.1 (LED_A)
- new net POOL_LINE: J5.3 (POOL), U20.2 (LED_K)
- new net REMOTE_POOL_SENSE: C3.1 (A), R4.2 (B), U20.4 (COLLECTOR)
- new net REMOTE_SPA_SENSE: C2.1 (A), R3.2 (B), U19.4 (COLLECTOR)
- new net SPA_LED_A: R1.2 (B), U19.1 (LED_A)
- new net SPA_LINE: J5.1 (SPA), U19.2 (LED_K)
- no-connect marks 0 -> 9
Other:
- note added: "DRY-CONTACT SENSE CIRCUIT: ISO_REMOTE_5V wets Pool/Spa contacts through R1/R2 and U19/U20 LEDs. COMMON_LINE is the isolated return. U19/U20 logic outputs are pulled up to +3V3 and filtered before firmware resolves Pool/Spa/Off/fault."
